File: AstraBeamLEDPCB/AstraBeamLED.kicad_pcb (KiCad board)
At the start: 2 copper layers, 75 x 55 mm, 20 parts

Commit message: Update for render
Other:
- board text added: "JLCJLCJLCJLC"
- board text removed: "REmove this"
Changed lines of the file:
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@@
 			(at 0 6.35 0)
 			(layer "F.Fab")
+			(hide yes)
 			(effects
 				(font
@@
 			(at 0 6.35 0)
 			(layer "F.Fab")
+			(hide yes)
 			(effects
 				(font
@@
 		(at 150 100 180)
 		(property "Reference" "D1"
-			(at 0 -4.25 0)
+			(at 0.000444 0.00122 0)
 			(layer "F.SilkS")
-			(hide yes)
 			(effects
 				(font
@@
 			(at 0 7 0)
 			(layer "F.Fab")
+			(hide yes)
 			(effects
 				(font
@@
 			(layer "F.Fab")
 		)
-		(fp_text user "${REFERENCE}"
-			(at 0 5 0)
-			(layer "F.Fab")
-			(effects
-				(font
-					(size 1 1)
-					(thickness 0.15)
-				)
-			)
-		)
 		(dimension
 			(type aligned)
@@
 			(at 0 6.35 0)
 			(layer "F.Fab")
+			(hide yes)
 			(effects
 				(font
@@
 			(at 0 6.35 0)
 			(layer "F.Fab")
+			(hide yes)
 			(effects
 				(font
@@
 			(at 0 6.35 0)
 			(layer "F.Fab")
+			(hide yes)
 			(effects
 				(font
@@
 			(at 0 6.35 0)
 			(layer "F.Fab")
+			(hide yes)
 			(effects
 				(font
@@
 			(at 0 6.35 0)
 			(layer "F.Fab")
+			(hide yes)
 			(effects
 				(font
@@
 			(at 0 6.35 0)
 			(layer "F.Fab")
+			(hide yes)
 			(effects
 				(font
@@
 		(layer "User.8")
 	)
-	(gr_text "REmove this"
-		(at 72.75 44.5 0)
-		(layer "User.8")
+	(gr_text "JLCJLCJLCJLC"
+		(at 150 121 0)
+		(layer "F.SilkS")
 		(effects
 			(font
@@
 				(thickness 0.15)
 			)
-			(justify left bottom)
 		)
 	)
@@
 			(xy 150 100) (xy 166.444621 94.014647)
 		)
-		(height -0.631961)
+		(height -0.001298)
 		(gr_text "17.5 mm"
-			(at 157.612845 95.332828 20.00000332)
+			(at 157.828544 95.925457 20.00000332)
 			(layer "User.8")
 			(effects
@@
 		(style
 			(thickness 0.15)
-			(arrow_length 1.27)
+			(arrow_length 0.5)
 			(text_position_mode 0)
 			(extension_height 0.58642)
@@
 		(style
 			(thickness 0.15)
-			(arrow_length 1.27)
+			(arrow_length 0.5)
 			(text_position_mode 0)
 			(extension_height 0.58642)
@@
 			(xy 178.25 120.75) (xy 180.75 120.75)
 		)
-		(height -5.75)
+		(height -3.75)
 		(gr_text "2.5 mm"
-			(at 179.5 113.85 0)
+			(at 179.5 115 0)
 			(layer "User.8")
 			(effects
@@
 		(style
 			(thickness 0.15)
-			(arrow_length 1.27)
-			(text_position_mode 0)
+			(arrow_length 0.5)
+			(text_position_mode 2)
 			(extension_height 0.58642)
 			(extension_offset 0.5) keep_text_aligned)
@@
 		(style
 			(thickness 0.15)
-			(arrow_length 0.4)
+			(arrow_length 0.5)
 			(text_position_mode 0)
 			(extension_height 0.58642)
@@
 		(style
 			(thickness 0.15)
-			(arrow_length 1.27)
+			(arrow_length 0.5)
 			(text_position_mode 0)
 			(extension_height 0.58642)
@@
 		(layer "User.8")
 		(pts
-			(xy 150 100) (xy 156 98)
+			(xy 150 100) (xy 153.25 100)
 		)
 		(gr_text "20deg"
-			(at 159.25 98 0)
+			(at 156.25 100 0)
 			(layer "User.8")
 			(effects
@@
 		(style
 			(thickness 0.15)
-			(arrow_length 1.27)
+			(arrow_length 0.5)
 			(text_position_mode 0)
 			(text_frame 0)
@@
 		(leader_length 3.81)
 		(gr_text "R 2.5 mm"
-			(at 158.25 75 0)
+			(at 161 75 0)
 			(layer "User.8")
 			(effects
@@
 		(style
 			(thickness 0.15)
-			(arrow_length 1.27)
+			(arrow_length 0.5)
 			(text_position_mode 0)
 			(extension_offset 0.5) keep_text_aligned)
@@
 		(style
 			(thickness 0.15)
-			(arrow_length 1.27)
+			(arrow_length 0.5)
 			(text_position_mode 0)
 			(extension_offset 0.5) keep_text_aligned)
@@
 		(style
 			(thickness 0.15)
-			(arrow_length 1.27)
+			(arrow_length 0.5)
 			(text_position_mode 0)
 			(extension_offset 0.5) keep_text_aligned)
@@
 		(leader_length 3.81)
 		(gr_text "R 1 mm"
-			(at 138 100 0)
+			(at 138.39 100 0)
 			(layer "User.8")
 			(effects
@@
 		(style
 			(thickness 0.15)
-			(arrow_length 1.27)
+			(arrow_length 0.5)
 			(text_position_mode 0)
-			(extension_offset 0.5) keep_text_aligned)
+			(extension_offset 0.05) keep_text_aligned)
 	)
 	(dimension
@@
 		(style
 			(thickness 0.15)
-			(arrow_length 1.27)
+			(arrow_length 0.5)
 			(text_position_mode 0)
 			(extension_offset 0.5) keep_text_aligned)
@@
 		(style
 			(thickness 0.15)
-			(arrow_length 1.27)
+			(arrow_length 0.5)
 			(text_position_mode 0)
 			(extension_offset 0.5) keep_text_aligned)
